File: Cad Files/REM PI FC.kicad_pcb (KiCad board)
At the start: 2 copper layers, 85 x 56 mm, 20 parts, among them J1 GPIO, J2 RJ45_LED_Shielded, J3 RJ45_LED_Shielded, J4 RJ45_LED_Shielded, J5 RJ45_LED_Shielded, K1-AD1 Songle SRD-5VDC-SL-C, K2-Enable1 Songle SRD-5VDC-SL-C, Q1 PN2222A, Q2 PN2222A

Commit message: Improved static resistance
Routing:
- net GND: track 133.6 -> 178.9 mm, vias 12 -> 19
- net +3V3: track 21.6 -> 0.00 mm
- net Net-(J2-Pad3): track 143.6 -> 145.6 mm
- net Net-(J2-Pad2): track 133.8 -> 134.7 mm
