File: Cad Files/REM PI FC.kicad_sch (KiCad schematic)
At the start: 21 parts, among them J1 GPIO, J2 RJ45_LED_Shielded, J3 RJ45_LED_Shielded, J4 RJ45_LED_Shielded, J5 RJ45_LED_Shielded, K1-AD1 Songle SRD-5VDC-SL-C, K2-Enable1 Songle SRD-5VDC-SL-C, Q1 PN2222A, Q2 PN2222A, U1 CAT24C256

Commit message: Improved static resistance
Other:
- note removed: "Additional pin functions: https://pinout.xyz/"
- company: (none) -> Designed By Matthew Beaudin
Changed lines of the file:
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@@
 	(title_block
 		(title "REM Pi FC")
-		(date "15 nov 2012")
-	)
-	(text "Additional pin functions:\nhttps://pinout.xyz/"
-		(exclude_from_sim no)
-		(at 179.07 180.34 0)
-		(effects
-			(font
-				(size 1.27 1.27)
-			)
-			(justify left bottom)
-		)
+		(date "10/9/2026")
+		(rev "1.2")
+		(company "Designed By Matthew Beaudin")
 	)
 	(text "ID_SD and ID_SC PINS:\nThese pins are reserved for HAT ID EEPROM.\n\nAt boot time this I2C interface will be\ninterrogated to look for an EEPROM\nthat identifes the attached board and\nallows automagic setup of the GPIOs\n(and optionally, Linux drivers).\n\nBridging JP1 enables write protection.\n\nDO NOT USE these pins for anything other\nthan attaching an I2C ID EEPROM. Leave\nunconnected if ID EEPROM not required."
@@
 	)
 	(junction
-		(at 186.69 99.06)
-		(diameter 0)
-		(color 0 0 0 0)
-	)
-	(junction
 		(at 203.2 46.99)
 		(diameter 0)
@@
 	)
 	(junction
+		(at 186.69 99.06)
+		(diameter 0)
+		(color 0 0 0 0)
+	)
+	(junction
 		(at 132.08 95.25)
 		(diameter 0)
@@
 		(in_pos_files yes)
 		(dnp no)
-		(fields_autoplaced yes)
 		(property "Reference" "#PWR08"
 			(at 207.01 106.68 0)
@@
 		)
 		(property "Value" "+5V"
-			(at 199.39 106.6799 90)
+			(at 202.692 104.14 90)
 			(show_name no)
 			(do_not_autoplace no)
@@
 		(dnp no)
 		(property "Reference" "R6"
-			(at 125.73 24.13 90)
+			(at 135.382 23.876 90)
 			(show_name no)
 			(do_not_autoplace no)
@@
 		)
 		(property "Value" "R30"
-			(at 128.27 24.13 90)
+			(at 137.922 24.13 90)
 			(show_name no)
 			(do_not_autoplace no)
